File: ai03-pcb-guide.kicad_sch (KiCad schematic)
At the start: 0 parts

Commit message: Add submodules
Parts:
- added F1: 500mA, symbol Device:Polyfuse_Small
- added U1: Seeed Studio XIAO RP2040, Seeed Studio XIAO Series Library:XIAO-Generic-Thruhole-14P-2.54-21X17.8MM, symbol Seeed_Studio_XIAO_Series:Seeed Studio XIAO SAMD21
- added USB1: Molex-0548190589, symbol random-keyboard-parts:Molex-0548190589
Connections:
- new net +5V: F1.2
- new net D+: USB1.3 (D+)
- new net D-: USB1.4 (D-)
- new net GND: U1.13 (GND), USB1.1 (GND)
- new net VCC: F1.1, U1.14 (5V), USB1.5 (VBUS)

Commit message: more commit
Parts:
- removed U1: Seeed Studio XIAO RP2040, Seeed Studio XIAO Series Library:XIAO-Generic-Thruhole-14P-2.54-21X17.8MM, symbol Seeed_Studio_XIAO_Series:Seeed Studio XIAO SAMD21
- added D1, D10, D2, D3, D4, D5, D6, D7, D8, D9: D_Small, Diode_SMD:D_SOD-123, symbol Device:D_Small
- added MX1, MX10, MX2, MX3, MX4, MX5, MX6, MX7, MX8, MX9: MX-NoLED, MX_Alps_Hybrid:MX-1U-NoLED, symbol MX_Alps_Hybrid:MX-NoLED
- added U1: MOUDLE-SEEEDUINO-XIAO, XIAO_PCB:MOUDLE14P-2.54-21X17.8MM, symbol MOUDLE-SEEEDUINO-XIAO:MOUDLE-SEEEDUINO-XIAO
- F1: footprint (none) -> Fuse:Fuse_1206_3216Metric
- USB1: footprint (none) -> random-keyboard-parts:Molex-0548190589
Connections:
- net GND: now also U1.13 (GND)
- net VCC: now also U1.14 (5V)
- new net: D4.2 (A), MX4.2 (ROW)
- new net: D5.2 (A), MX5.2 (ROW)
- new net: D2.2 (A), MX2.2 (ROW)
- new net: D6.2 (A), MX6.2 (ROW)
- new net: D1.2 (A), MX1.2 (ROW)
- new net: D10.2 (A), MX10.2 (ROW)
- new net: D7.2 (A), MX7.2 (ROW)
- new net: D9.2 (A), MX9.2 (ROW)
- new net: D3.2 (A), MX3.2 (ROW)
- new net: D8.2 (A), MX8.2 (ROW)
- new net COL 0: MX1.1 (COL), MX3.1 (COL)
- new net COL 1: MX2.1 (COL), MX4.1 (COL)
- new net COL 2: MX10.1 (COL), MX8.1 (COL)
- new net COL 3: MX5.1 (COL), MX9.1 (COL)
- new net COL 4: MX6.1 (COL), MX7.1 (COL)
- new net ROW 0: D1.1 (K), D2.1 (K), D5.1 (K), D6.1 (K)
- new net ROW 1: D3.1 (K), D7.1 (K)
- new net ROW 2: D4.1 (K), D8.1 (K), D9.1 (K)
- new net ROW 3: D10.1 (K)

Commit message: i commit
Parts:
- added Brd1: SSD1306, SSD1306:128x64OLED, symbol SSD1306-128x64_OLED:SSD1306
Connections:
- net GND: now also Brd1.1 (GND)
- net VCC: now also Brd1.2 (VCC)
- net at U1.5 (PA8_A4_D4_SDA): now also Brd1.4 (SDA)
- net at U1.6 (PA9_A5_D5_SCL): now also Brd1.3 (SCL)

Commit message: second commit of the day!
Parts:
- removed Brd1: SSD1306, SSD1306:128x64OLED, symbol SSD1306-128x64_OLED:SSD1306
- removed F1: 500mA, Fuse:Fuse_1206_3216Metric, symbol Device:Polyfuse_Small
- removed USB1: Molex-0548190589, random-keyboard-parts:Molex-0548190589, symbol random-keyboard-parts:Molex-0548190589
- added OL1: OLED, kbd:OLED, symbol kbd:OLED
Connections:
- net GND: now also OL1.4 (GND)
- net VCC: now also OL1.3 (VCC)
- net at U1.5 (PA8_A4_D4_SDA): now also OL1.1 (SDA)
- net at U1.6 (PA9_A5_D5_SCL): now also OL1.2 (SCL)

Commit message: yay
Connections:
- net COL 0: now also U1.11 (PA6_A10_D10_MOSI)
- net COL 1: now also U1.10 (PA5_A9_D9_MISO)
- net COL 2: now also U1.9 (PA7_A8_D8_SCK)
- net COL 3: now also U1.8 (PB09_A7_D7_RX)
- net COL 4: now also U1.7 (PB08_A6_D6_TX)
- net ROW 0: now also U1.4 (PA11_A3_D3)
- net ROW 1: now also U1.3 (PA10_A2_D2)
- net ROW 2: now also U1.2 (PA4_A1_D1)
- net ROW 3: now also U1.1 (PA02_A0_D0)

Commit message: a commit
Parts:
- MX1, MX10, MX2, MX3, MX4, MX5, MX6, MX7, MX8, MX9: footprint MX_Alps_Hybrid:MX-1U-NoLED -> Button_Switch_Keyboard:SW_Cherry_MX_1.00u_PCB
Changed lines of the file:
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@@
 			)
 		)
-		(property "Footprint" "MX_Alps_Hybrid:MX-1U-NoLED"
+		(property "Footprint" "Button_Switch_Keyboard:SW_Cherry_MX_1.00u_PCB"
 			(at 71.755 116.205 0)
 			(effects
@@
 			)
 		)
-		(property "Footprint" "MX_Alps_Hybrid:MX-1U-NoLED"
+		(property "Footprint" "Button_Switch_Keyboard:SW_Cherry_MX_1.00u_PCB"
 			(at 84.455 116.205 0)
 			(effects
@@
 			)
 		)
-		(property "Footprint" "MX_Alps_Hybrid:MX-1U-NoLED"
+		(property "Footprint" "Button_Switch_Keyboard:SW_Cherry_MX_1.00u_PCB"
 			(at 33.655 128.905 0)
 			(effects
@@
 			)
 		)
-		(property "Footprint" "MX_Alps_Hybrid:MX-1U-NoLED"
+		(property "Footprint" "Button_Switch_Keyboard:SW_Cherry_MX_1.00u_PCB"
 			(at 84.455 128.905 0)
 			(effects
@@
 			)
 		)
-		(property "Footprint" "MX_Alps_Hybrid:MX-1U-NoLED"
+		(property "Footprint" "Button_Switch_Keyboard:SW_Cherry_MX_1.00u_PCB"
 			(at 46.355 116.205 0)
 			(effects
@@
 			)
 		)
-		(property "Footprint" "MX_Alps_Hybrid:MX-1U-NoLED"
+		(property "Footprint" "Button_Switch_Keyboard:SW_Cherry_MX_1.00u_PCB"
 			(at 59.055 154.305 0)
 			(effects
@@
 			)
 		)
-		(property "Footprint" "MX_Alps_Hybrid:MX-1U-NoLED"
+		(property "Footprint" "Button_Switch_Keyboard:SW_Cherry_MX_1.00u_PCB"
 			(at 59.055 141.605 0)
 			(effects
@@
 			)
 		)
-		(property "Footprint" "MX_Alps_Hybrid:MX-1U-NoLED"
+		(property "Footprint" "Button_Switch_Keyboard:SW_Cherry_MX_1.00u_PCB"
 			(at 71.755 141.605 0)
 			(effects
@@
 			)
 		)
-		(property "Footprint" "MX_Alps_Hybrid:MX-1U-NoLED"
+		(property "Footprint" "Button_Switch_Keyboard:SW_Cherry_MX_1.00u_PCB"
 			(at 46.355 141.605 0)
 			(effects
@@
 			)
 		)
-		(property "Footprint" "MX_Alps_Hybrid:MX-1U-NoLED"
+		(property "Footprint" "Button_Switch_Keyboard:SW_Cherry_MX_1.00u_PCB"
 			(at 33.655 116.205 0)
 			(effects
