File: ai03-pcb-guide.kicad_pcb (KiCad board)
At the start: 2 copper layers, 38.1 x 59.5 mm, 23 parts, among them U1 MOUDLE-SEEEDUINO-XIAO

Commit message: i commit
Parts:
- added Brd1: SSD1306, SSD1306:128x64OLED, F.Cu at (128.6, 21.4)
- U1: moved to B.Cu
- moved U1 104.4 mm to (111.1, 68.3), turned to 180 degrees
Connections:
- U1 pad 5: unconnected-(U1-PA8_A4_D4_SDA-Pad5) -> Net-(Brd1-SDA)
- U1 pad 6: unconnected-(U1-PA9_A5_D5_SCL-Pad6) -> Net-(Brd1-SCL)
Other:
- board size 38.1 x 59.5 mm -> 95.2 x 76.2 mm

Commit message: second commit of the day!
Parts:
- removed Brd1: SSD1306, SSD1306:128x64OLED
- removed F1: 500mA, Fuse:Fuse_1206_3216Metric
- removed USB1: Molex-0548190589, random-keyboard-parts:Molex-0548190589
- added OL1: OLED, kbd:OLED, F.Cu at (145.6, 68.3)
- moved U1 0.79 mm to (111.1, 69.1), turned to 0 degrees
Routing:
- net ROW 0: track 0.00 -> 87.9 mm
- net ROW 1: track 0.00 -> 76.8 mm
- net Net-(OL1-SCL): track 0.00 -> 42.5 mm
- net COL 3: track 0.00 -> 39.7 mm
- net ROW 2: track 0.00 -> 39.3 mm
- net Net-(OL1-SDA): track 0.00 -> 38.9 mm
- net COL 1: track 0.00 -> 37.2 mm
- net GND: track 0.00 -> 31.6 mm
- net VCC: track 0.00 -> 29.1 mm
- net COL 4: track 0.00 -> 18.1 mm
- net COL 2: track 0.00 -> 18.1 mm
- net COL 0: track 0.00 -> 18.1 mm
- net Net-(D4-A): track 0.00 -> 6.82 mm
- net Net-(D3-A): track 0.00 -> 6.79 mm
- net Net-(D10-A): track 0.00 -> 6.62 mm
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Other:
- outline, holes or cut-outs redrawn

Commit message: yay
Connections:
- U1 pad 1: unconnected-(U1-PA02_A0_D0-Pad1) -> COL 0
- U1 pad 10: unconnected-(U1-PA5_A9_D9_MISO-Pad10) -> ROW 2
- U1 pad 11: unconnected-(U1-PA6_A10_D10_MOSI-Pad11) -> ROW 3
- U1 pad 2: unconnected-(U1-PA4_A1_D1-Pad2) -> COL 1
- U1 pad 3: unconnected-(U1-PA10_A2_D2-Pad3) -> COL 2
- U1 pad 4: unconnected-(U1-PA11_A3_D3-Pad4) -> COL 3
- U1 pad 7: unconnected-(U1-PB08_A6_D6_TX-Pad7) -> COL 4
- U1 pad 8: unconnected-(U1-PB09_A7_D7_RX-Pad8) -> ROW 0
- U1 pad 9: unconnected-(U1-PA7_A8_D8_SCK-Pad9) -> ROW 1
Routing:
- net COL 3: track 39.7 -> 108.1 mm, vias 0 -> 4
- net COL 4: track 18.1 -> 82.6 mm, vias 0 -> 2
- net ROW 3: track 0.00 -> 63.5 mm, vias 0 -> 2
- net ROW 2: track 39.3 -> 82.9 mm
- net COL 0: track 18.1 -> 59.0 mm, vias 0 -> 1
- net COL 1: track 37.2 -> 59.6 mm
- net COL 2: track 18.1 -> 32.5 mm, vias 0 -> 1
- net ROW 1: track 76.8 -> 86.7 mm, vias 0 -> 2
- net ROW 0: track 87.9 -> 93.3 mm
Other:
- board size 95.2 x 76.2 mm -> 100 x 81 mm
- board text added: "HeartPad"

Commit message: a commit
Parts:
- MX1, MX10, MX2, MX3, MX4, MX5, MX6, MX7, MX8, MX9: footprint MX_Alps_Hybrid:MX-1U-NoLED -> Button_Switch_Keyboard:SW_Cherry_MX_1.00u_PCB; moved to B.Cu
- moved MX3 5.68 mm to (86.4, 63.2), turned to 180 degrees
- moved MX5 5.68 mm to (143.5, 44.1), turned to 180 degrees
- moved MX9 5.68 mm to (143.5, 82.2), turned to 180 degrees
- moved MX1 5.68 mm to (86.4, 44.1), turned to 180 degrees
- moved MX10 5.68 mm to (124.5, 101.3), turned to 180 degrees
- moved MX2 5.68 mm to (105.4, 44.1), turned to 180 degrees
- moved MX4 5.68 mm to (105.4, 82.2), turned to 180 degrees
- moved MX7 5.68 mm to (162.6, 63.2), turned to 180 degrees
- moved MX8 5.68 mm to (124.5, 82.2), turned to 180 degrees
- moved MX6 5.68 mm to (162.6, 44.1), turned to 180 degrees
- moved D10 0.32 mm to (135.2, 106.3)
- moved D9 0.32 mm to (154.3, 87.2)
- moved D7 0.31 mm to (173.3, 68.2)
- moved D2 0.31 mm to (116.2, 49.2)
- moved D1 0.31 mm to (97.2, 49.1)
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Connections:
- U1 pad 1: COL 0 -> ROW 3
- U1 pad 10: ROW 2 -> COL 1
- U1 pad 11: ROW 3 -> COL 0
- U1 pad 2: COL 1 -> ROW 2
- U1 pad 3: COL 2 -> ROW 1
- U1 pad 4: COL 3 -> ROW 0
- U1 pad 8: ROW 0 -> COL 3
- U1 pad 9: ROW 1 -> COL 2
Routing:
- net ROW 2: track 82.9 -> 55.8 mm
- net ROW 0: track 93.3 -> 119.5 mm, vias 0 -> 2
- net COL 2: track 32.5 -> 56.7 mm, vias 1 -> 2
- net COL 1: track 59.6 -> 46.3 mm, vias 0 -> 1
- net COL 0: track 59.0 -> 46.0 mm, vias 1 -> 0
- net ROW 3: track 63.5 -> 51.4 mm
- net ROW 1: track 86.7 -> 81.8 mm, vias 2 -> 0
- net COL 4: track 82.6 -> 86.5 mm, vias 2 -> 0
- net COL 3: track 108.1 -> 106.2 mm, vias 4 -> 5
- net Net-(D2-A): track 6.62 -> 4.80 mm
- net Net-(D6-A): track 6.62 -> 4.81 mm
- net Net-(D5-A): track 6.62 -> 4.81 mm
- net Net-(D4-A): track 6.62 -> 4.81 mm
- net Net-(D8-A): track 6.62 -> 4.81 mm
- net Net-(D1-A): track 6.59 -> 4.78 mm
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
Commit message: added kitty
Parts:
- added G***: LOGO, kitty:kitty, B.Cu at (133.5, 69.0)
